File: schematic/Dram-Tester-x1x4-lcd.kicad_sch (KiCad schematic)
At the start: 56 parts, among them IC1 TC7660S, J1 MJ-179PH, J2 PS, SW1 DTS-63N-V, SW2 SS12SDP2, SW3 SS22SDP2, U1 Arduino Nano, U2 MT3608 DCDC Module, U3 I2C OLED Screen 0.91 128x32, U4 (AL12832AWWB-H-U02)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

Commit message: Schematic modified
回路図を修正
Schematic modified.
積層セラミックコンデンサのピッチを2.5mmに変更
Changed pitch of MLCC to 2.5 mm.
未実装の5V-DCDCモジュールを削除
Remove unmounted 5V-DCDC module
重複していたパスコンを削除
Removed duplicated bypass capacitor.
47μFの電解コンデンサを10μFに変更
47uF ELC changed to 10uF.
チャージポンプの品番をTC7660SからTJ7660に変更
The part number of the charge pump was changed from TC7660S to TJ7660.
その他細かな修正
Other minor modifications.
Parts:
- removed C8: 0.1u, Capacitor_THT:C_Disc_D4.3mm_W1.9mm_P5.00mm, symbol Device:C_Small
- removed J2: PS, Connector_PinHeader_2.54mm:PinHeader_1x02_P2.54mm_Vertical, symbol Connector_Generic:Conn_01x02
- removed JP2: 5V, Jumper:SolderJumper-2_P1.3mm_Bridged_RoundedPad1.0x1.5mm, symbol Jumper:Jumper_2_Bridged
- removed U5: (AE-XCL103-5V0), ProjectLibrary:DIP6_300mil_FineLongPad_No3D, symbol ProjectLibrary:AE-XCL103_Horizontal
- added U6: (PDT006-9V), Connector_PinHeader_2.54mm:PinHeader_1x02_P2.54mm_Vertical, symbol Connector_Generic:Conn_01x02
- C1, C2, C3, C4: footprint Capacitor_THT:C_Disc_D4.3mm_W1.9mm_P5.00mm -> Capacitor_THT:C_Disc_D3.4mm_W2.1mm_P2.50mm
- C6: value 47u -> 10u
- IC1: value TC7660S -> TJ7660
- JP1: value Pin Header 1x3pin -> LEDTYP
- JP2: renamed from JP5; value A9EN -> (A9EN)
- LED2: value Green -> SCKTPW
- R19: value 47 -> (47)
- U3: value I2C OLED Screen 0.91 128x32 -> I2C OLED Screen 0.91inch 128x32dot
- renumbered C9 to C8, J1 to CN1, JP3 to J1, JP4 to J2
Connections:
- net SOCKET_PS is gone; now on net SOCKET_5V: SW3.1 (NC_1), U2.1 (VIN+)
- net +5V: now also C4.2; no longer C4.1
- net -5V: now also C1.1; no longer C1.2
- net GND: now also C1.2, C4.1, U6.2 (Pin_2); no longer C1.1, C4.2
- net NPPS: now also U6.1 (Pin_1)
- no-connect marks 12 -> 10
Other:
- title: 1&4 bit support standalone DRAM tester with display. -> 1bit and 4bit support standalone DRAM tester with display
